File: hardware/prototype7_smd/edrumulus.kicad_pcb (KiCad board)
At the start: 2 copper layers, 200 x 100 mm, 124 parts, among them J1 Hi-Hat, J10 MIDI-IN, J11 MIDI-OUT, J12 Snare, J13 Snare, J14 Kick, J15 Conn_01x02_Socket, J16 Conn_01x02_Socket, J17 Conn_01x04, J2 Snare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

Commit message: Fix routing
Routing:
- net AN_HH_RING: track 74.0 -> 93.3 mm, vias 1 -> 2
- net +3.3V: track 564.2 -> 578.8 mm
- net AN_AUX3_TIP: track 75.2 -> 69.5 mm, vias 1 -> 2
- net AN_AUX1_RING: track 104.1 -> 108.8 mm
- net AN_SNARE_TIP: track 107.9 -> 111.4 mm
- net AN_KICK_TIP: track 78.7 -> 82.1 mm
- net AN_SNARE_RING: track 118.1 -> 120.1 mm
- net GPIO_BRD_ID1: track 1025.5 -> 1023.6 mm
- net AN_RIDE_RING: track 79.2 -> 80.9 mm
- net AN_CRASH_RING: track 85.2 -> 86.9 mm
- net AN_TOM2_TIP: track 40.8 -> 42.4 mm
- net AN_AUX2_RING: track 80.5 -> 82.0 mm
- net HI-HAT-RING: track 63.5 -> 64.7 mm
- net Net-(D7-A): track 33.1 -> 34.2 mm
- net Net-(J16-Pin_1): track 78.2 -> 79.4 mm
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- added copper zone on B.Cu, net AN_AUX2_RING
- removed copper zone on B.Cu, net GPIO_BRD_ID1
Other:
- board text added: "EDrumulus ESP32-S3 P7"
